File: USART.kicad_pcb (KiCad board)
At the start: 2 copper layers, 85 x 65 mm, 63 parts, among them X1 USART TTL, X2 Conn_01x10, X3 Power, X4 Address, X5 Data, X6 Mode, X7 Control, X8 Clock

Commit message: Update+fix
- Replaced the standard logic oscillator with a monolithic quartz oscillator;
- Fixed the 'CLK' source of the 580VV51 (8251);
- Connected the reset signal of the 580VV51 (8251).

- Заменен генератор на стандартной логике на монолитный кварцевый генератор;
- Исправлен источник 'CLK' у 580ВВ51 (8251);
- Подключен сигнал сброса у 580ВВ51 (8251).
Parts:
- removed the C1 at (92.0, 121.8)
- removed C13: 10p, Capacitor_SMD:C_0805_2012Metric_Pad1.18x1.45mm_HandSolder
- removed the C2 at (93.0, 128.3)
- removed the DD1 at (93.0, 116.7)
- removed the DD3 at (75.2, 136.8)
- removed R5, R6: 1k, Resistor_SMD:R_0805_2012Metric_Pad1.20x1.40mm_HandSolder
- R3: value 330 -> 1k
- R4: value 330 -> 0
- ZQ1: value 4.9152MHz -> 2457,6 kHz; footprint Crystal:Crystal_HC49-U_Vertical -> Oscillator:Oscillator_DIP-8_LargePads
- moved C8 17.2 mm to (84.1, 116.1), turned to 90 degrees
- moved ZQ1 14.8 mm to (84.1, 127.8)
- moved C7 9.18 mm to (84.1, 123.5), turned to -90 degrees
- moved R4 8.85 mm to (87.5, 127.8), turned to 180 degrees
- moved R3 7.81 mm to (80.8, 127.8)
- renumbered C9 to C1, C4 to C10, C10 to C2, C11 to C3, C12 to C4, C3 to C9, DD5 to DD1, DD6 to DD3, JP25 to JP1, JP16 to JP10, JP21 to JP11, JP9 to JP12, JP22 to JP13, JP10 to JP14, JP23 to JP15, JP11 to JP16, JP24 to JP17, JP12 to JP18, JP5 to JP19, JP26 to JP2, JP6 to JP20, JP7 to JP21, JP8 to JP22, JP1 to JP23, JP2 to JP24, JP3 to JP25, JP4 to JP26, JP17 to JP3, JP13 to JP4, JP18 to JP5, JP14 to JP6, JP19 to JP7, JP15 to JP8, JP20 to JP9, R2 to R1, R1 to R2, X3 to X1, X4 to X2, X5 to X3, X6 to X4, X7 to X5, X8 to X6, X2 to X7, X1 to X8
Connections:
- DD3 pad 20: /USART_OSC -> /Single_BCLK
- R3 pad 1: Net-(C13-Pad2) -> +5
- R3 pad 2: Net-(DD3-Pad2) -> Net-(ZQ1-EN)
- R4 pad 1: Net-(DD3-Pad2) -> GND
- R4 pad 2: Net-(DD3-Pad4) -> Net-(ZQ1-EN)
- X5 pad 10: /RESOUT -> /RESET
- ZQ1 pad 1: Net-(C13-Pad1) -> Net-(ZQ1-EN)
Routing:
- net /RESET: track 0.00 -> 54.3 mm, vias 0 -> 3
- net /Single_BCLK: track 0.00 -> 38.4 mm, vias 0 -> 3
- net +5: track 283.5 -> 247.7 mm
- net /USART_OSC: track 35.6 -> 0.00 mm, vias 4 -> 0
- net Net-(DD1A-C): track 22.2 -> 0.00 mm
- net Net-(DD1A-Q): track 18.5 -> 0.00 mm, vias 1 -> 0
- net Net-(DD1A-D): track 16.3 -> 0.00 mm
- net /~{BUSEN}: track 119.0 -> 104.3 mm
- net /PIT_OSC: track 56.0 -> 46.5 mm
- net Net-(DD3-Pad4): track 9.48 -> 0.00 mm
- net Net-(DD3-Pad2): track 7.48 -> 0.00 mm
- net Net-(C13-Pad2): track 5.08 -> 0.00 mm
- net Net-(ZQ1-EN): track 0.00 -> 4.69 mm
- net Net-(DD1A-~{R}): track 3.88 -> 0.00 mm
- net Net-(DD1A-~{S}): track 2.70 -> 0.00 mm
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Other:
- board text added: "2457,6 kHz"
- board text added: "BCLK"
- board text added: "OSC_TTL"
- board text added: "RESOUT"
- board text added: "v.1.2 03/12/2025"
- board text added: "~{BUSEN}"
- board text added: "~{STSTB}"
- board text removed: "555ЛН1"
- board text removed: "555ТМ2"
- board text removed: "v.1.1 24/11/2025"

Commit message: Add files via upload
Changed IRQ bus pin's

Изменены пины шины IRQ
Parts:
- ZQ1: value 2457,6 kHz -> 1843,2 kHz
- moved JP17 17.8 mm to (144.3, 90.3)
- moved JP3 17.8 mm to (126.5, 90.3)
- moved JP15 12.7 mm to (141.7, 90.3)
- moved JP5 12.7 mm to (129.0, 90.3)
- moved JP13 7.62 mm to (139.2, 90.3)
- moved JP7 7.62 mm to (131.6, 90.3)
- moved JP11 2.54 mm to (136.7, 90.3)
- moved JP9 2.54 mm to (134.1, 90.3)
Connections:
- X7 pad 2: /IRQ0 -> /IRQ7
- X7 pad 3: /IRQ1 -> /IRQ6
- X7 pad 4: /IRQ2 -> /IRQ5
- X7 pad 5: /IRQ3 -> /IRQ4
- X7 pad 6: /IRQ4 -> /IRQ3
- X7 pad 7: /IRQ5 -> /IRQ2
- X7 pad 8: /IRQ6 -> /IRQ1
- X7 pad 9: /IRQ7 -> /IRQ0
Other:
- board text added: "1843,2 kHz"
- board text added: "HLDA"
- board text added: "HRQ"
- board text added: "INT"
- board text added: "INTE"
- board text added: "WAIT"
- board text added: "XRDY"
- board text added: "~{INTA}"
- board text added: "~{RESIN}"
- board text removed: "2457,6 kHz"

Commit message: Add files via upload
Parts:
- added C7: 100n, Capacitor_SMD:C_0805_2012Metric_Pad1.18x1.45mm_HandSolder, B.Cu at (141.9, 109.0)
- moved R2 0.11 mm to (141.9, 111.0)
- renumbered C9 to C10, C10 to C11, C7 to C8, C8 to C9, JP11 to JP10, JP10 to JP11, JP13 to JP12, JP12 to JP13, JP15 to JP14, JP14 to JP15, JP17 to JP16, JP16 to JP17, JP5 to JP4, JP4 to JP5, JP7 to JP6, JP6 to JP7, JP9 to JP8, JP8 to JP9
Connections:
- net /INTE renamed /~{WRQ}
- net /RESET renamed /RESOUT
- net /Single_BCLK renamed /F2TTL
- net /Single_OSC_TTL renamed /OSC_TTL
Routing:
- net Net-(DD4-E3): track 2.29 -> 4.44 mm
- net /~{IOW}: track 44.2 -> 43.3 mm
- net /AB1: track 106.9 -> 107.8 mm
- net /USART_Tx: track 41.6 -> 42.5 mm
- net /AB0: track 103.9 -> 104.7 mm
- net /~{IOR}: track 57.7 -> 57.0 mm
- net /USART_~{CTS}: track 50.8 -> 51.5 mm
- net /DB5: track 43.9 -> 43.2 mm
- net /DB6: track 44.3 -> 43.7 mm
- net GND: vias 443 -> 466
Other:
- board text added: "F2TTL"
- board text added: "OSC"
- board text added: "~{CTS}-~{RTS}"
- board text added: "~{DSR}-~{DTR}"
- board text added: "~{MEMR}"
- board text added: "~{MEMW}"
- board text added: "~{WRQ}"
- board text removed: "BCLK"
- board text removed: "CTS-RTS"
- board text removed: "DSR-DTR"
- board text removed: "INTE"
- board text removed: "OSC_TTL"
